File: obj-89/obj-89.kicad_pcb (KiCad board)
At the start: 2 copper layers, 24 parts, among them J1 Power, J2 Conn_01x04_Male, J3 Conn_01x04_Male, J4 Conn_01x06_Male, SW1 KEY, SW2 KEY, SW3 KEY, SW4 KEY, SW5 KEY, SW6 KEY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

Commit message: update
unfinish
Parts:
- added REF: MountingHole_3.2mm_M3, Mounting_Holes:MountingHole_3.2mm_M3, F.Cu at (167.6, 129.5)
- added REF: MountingHole_3.2mm_M3, Mounting_Holes:MountingHole_3.2mm_M3, F.Cu at (167.6, 80.0)
- added REF: MountingHole_3.2mm_M3, Mounting_Holes:MountingHole_3.2mm_M3, F.Cu at (88.9, 80.0)
- added REF: MountingHole_3.2mm_M3, Mounting_Holes:MountingHole_3.2mm_M3, F.Cu at (88.9, 129.5)
- R1, R2, R3, R4, R5, R6: footprint Resistors_SMD:R_0201 -> Resistors_THT:R_Axial_DIN0207_L6.3mm_D2.5mm_P7.62mm_Horizontal
- moved J2 86.4 mm to (94.0, 115.6), turned to 180 degrees
- moved SW5 58.5 mm to (94.0, 83.8)
- moved J3 54.0 mm to (94.0, 96.5)
- moved SW1 50.3 mm to (94.0, 120.7)
- moved SW6 48.0 mm to (105.4, 83.8)
- moved SW2 45.8 mm to (105.4, 120.7)
- moved SW7 38.1 mm to (116.8, 83.8)
- moved J4 37.6 mm to (163.8, 110.5), turned to 180 degrees
- moved SW3 35.3 mm to (116.8, 120.7)
- moved SW8 29.3 mm to (128.3, 83.8)
- moved SW4 25.6 mm to (128.3, 120.7)
- moved D6 20.3 mm to (144.8, 85.1), turned to 180 degrees
- moved R6 20.0 mm to (149.9, 85.1)
- moved D1 19.2 mm to (142.2, 123.2)
- moved R1 18.2 mm to (149.9, 123.2)
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Routing:
- net Net-(D1-Pad1): track 0.00 -> 73.0 mm
- net Net-(D4-Pad2): track 0.00 -> 72.7 mm
- net Net-(J3-Pad4): track 0.00 -> 49.2 mm
- net Net-(J2-Pad4): track 0.00 -> 46.1 mm
- net Net-(J3-Pad3): track 0.00 -> 36.7 mm
- net Net-(J2-Pad3): track 0.00 -> 33.6 mm
- net Net-(J3-Pad2): track 0.00 -> 24.2 mm
- net Net-(J2-Pad2): track 0.00 -> 21.1 mm
- net Net-(J4-Pad6): track 0.00 -> 15.3 mm
- net Net-(J4-Pad1): track 0.00 -> 15.3 mm
- net Net-(J3-Pad1): track 0.00 -> 14.7 mm
- net Net-(J4-Pad5): track 0.00 -> 12.5 mm
- net Net-(J4-Pad2): track 0.00 -> 12.5 mm
- net Net-(J2-Pad1): track 0.00 -> 11.6 mm
- net Net-(J4-Pad4): track 0.00 -> 8.15 mm
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- added copper zone on B.Cu, net (none)
