File: obj-89/obj-89.sch (KiCad schematic (older format))
At the start: 24 parts, among them J1 Power, J2 Conn_01x04_Male, J3 Conn_01x04_Male, J4 Conn_01x06_Male, SW1 KEY, SW2 KEY, SW3 KEY, SW4 KEY, SW5 KEY, SW6 KEY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

Commit message: update
unfinish
Parts:
- R1, R2, R3, R4, R5, R6: footprint Resistors_SMD:R_0201 -> Resistors_THT:R_Axial_DIN0207_L6.3mm_D2.5mm_P7.62mm_Horizontal
Changed lines of the file:
@@
 F 0 "R1" V 3130 2900 50  0000 C CNN
 F 1 "R220" V 3050 2900 50  0000 C CNN
-F 2 "Resistors_SMD:R_0201" V 2980 2900 50  0001 C CNN
+F 2 "Resistors_THT:R_Axial_DIN0207_L6.3mm_D2.5mm_P7.62mm_Horizontal" V 2980 2900 50  0001 C CNN
 F 3 "" H 3050 2900 50  0001 C CNN
 	1    3050 2900
@@
 F 0 "R2" V 3130 3200 50  0000 C CNN
 F 1 "R220" V 3050 3200 50  0000 C CNN
-F 2 "Resistors_SMD:R_0201" V 2980 3200 50  0001 C CNN
+F 2 "Resistors_THT:R_Axial_DIN0207_L6.3mm_D2.5mm_P7.62mm_Horizontal" V 2980 3200 50  0001 C CNN
 F 3 "" H 3050 3200 50  0001 C CNN
 	1    3050 3200
@@
 F 0 "R3" V 3130 3500 50  0000 C CNN
 F 1 "R220" V 3050 3500 50  0000 C CNN
-F 2 "Resistors_SMD:R_0201" V 2980 3500 50  0001 C CNN
+F 2 "Resistors_THT:R_Axial_DIN0207_L6.3mm_D2.5mm_P7.62mm_Horizontal" V 2980 3500 50  0001 C CNN
 F 3 "" H 3050 3500 50  0001 C CNN
 	1    3050 3500
@@
 F 0 "R4" V 3130 3950 50  0000 C CNN
 F 1 "R220" V 3050 3950 50  0000 C CNN
-F 2 "Resistors_SMD:R_0201" V 2980 3950 50  0001 C CNN
+F 2 "Resistors_THT:R_Axial_DIN0207_L6.3mm_D2.5mm_P7.62mm_Horizontal" V 2980 3950 50  0001 C CNN
 F 3 "" H 3050 3950 50  0001 C CNN
 	1    3050 3950
@@
 F 0 "R5" V 3130 4250 50  0000 C CNN
 F 1 "R220" V 3050 4250 50  0000 C CNN
-F 2 "Resistors_SMD:R_0201" V 2980 4250 50  0001 C CNN
+F 2 "Resistors_THT:R_Axial_DIN0207_L6.3mm_D2.5mm_P7.62mm_Horizontal" V 2980 4250 50  0001 C CNN
 F 3 "" H 3050 4250 50  0001 C CNN
 	1    3050 4250
@@
 F 0 "R6" V 3130 4550 50  0000 C CNN
 F 1 "R220" V 3050 4550 50  0000 C CNN
-F 2 "Resistors_SMD:R_0201" V 2980 4550 50  0001 C CNN
+F 2 "Resistors_THT:R_Axial_DIN0207_L6.3mm_D2.5mm_P7.62mm_Horizontal" V 2980 4550 50  0001 C CNN
 F 3 "" H 3050 4550 50  0001 C CNN
 	1    3050 4550
