File: or-serial/or-serial.kicad_pcb (KiCad board)
At the start: 2 copper layers, 9 parts, among them J0 LC12S, J1 OLED, J2 GPS, J3-l1 speaker (left pins), J3-r1 speaker (right pins), J4 IR, J5-l1 Out(1), J5-r1 Out(2)

Commit message: re-update
Parts:
- added REF**: WireConnection_0-8mmDrill_ThinPad, Wire_Connections_Bridges:WireConnection_0.80mmDrill_ThinPad, F.Cu at (43.8, 75.6)
Routing:
- net GND: track 263.4 -> 277.7 mm
- net +3V3: track 171.8 -> 180.7 mm
- net +5V: track 77.9 -> 83.0 mm
- net Net-(J2-Pad2): track 39.4 -> 43.8 mm
- net Net-(J1-Pad6): track 28.7 -> 32.7 mm
- net Net-(J1-Pad4): track 27.2 -> 30.1 mm
- net Net-(J2-Pad3): track 48.6 -> 51.3 mm
- net Net-(J1-Pad3): track 28.1 -> 30.5 mm
- net Net-(J3-l1-Pad7): track 86.3 -> 88.1 mm
- net Net-(J3-l1-Pad8): track 92.9 -> 94.4 mm
- net Net-(J4-Pad3): track 87.8 -> 88.8 mm
Other:
- net class Default: trace_width 0.25 -> 1
- rule trace_min: 0.2 -> 1
