File: experiment/hole_dual/hole_dual.kicad_pcb (KiCad board)
At the start: 2 copper layers, 3 parts, among them J1 Conn_01x08, J2 Conn_01x08

Commit message: update
Parts:
- removed the REF** at (160.7, 129.5)
- added REF**: MountingHole_3.2mm_M3, Mounting_Holes:MountingHole_3.2mm_M3, F.Cu at (112.4, 127.6)
- added REF**: MountingHole_3.2mm_M3, Mounting_Holes:MountingHole_3.2mm_M3, F.Cu at (112.4, 100.3)
- added REF**: MountingHole_3.2mm_M3, Mounting_Holes:MountingHole_3.2mm_M3, F.Cu at (152.4, 100.3)
- added REF**: MountingHole_3.2mm_M3, Mounting_Holes:MountingHole_3.2mm_M3, F.Cu at (152.4, 127.6)
Routing:
- added copper zone on B.Cu, net (none)
- added copper zone on F.Cu, net (none)
Other:
- net class Default: clearance 0.2 -> 0.25; trace_width 0.25 -> 0.7; via_dia 0.6 -> 0.8; via_drill 0.4 -> 0.6
- rule trace_clearance: 0.2 -> 0.25
Changed lines of the file:
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@@
     (links 8)
     (no_connects 0)
-    (area 109.895 97.83 159.814286 134.71)
+    (area 102.792857 95.075 162.007143 132.925)
     (thickness 1.6)
     (drawings 4)
     (tracks 24)
     (zones 0)
-    (modules 3)
+    (modules 6)
     (nets 9)
   )
@@
   )
   (setup
-    (last_trace_width 0.25)
-    (trace_clearance 0.2)
+    (last_trace_width 0.7)
+    (trace_clearance 0.25)
     (zone_clearance 0.508)
     (zone_45_only no)
@@
     (segment_width 0.2)
     (edge_width 0.15)
-    (via_size 0.6)
-    (via_drill 0.4)
+    (via_size 0.8)
+    (via_drill 0.6)
     (via_min_size 0.4)
     (via_min_drill 0.3)
@@
     (pad_to_mask_clearance 0.2)
     (aux_axis_origin 0 0)
-    (visible_elements FFFFFF7F)
+    (visible_elements FFFFF77F)
     (pcbplotparams
       (layerselection 0x3ffff_80000001)
       (usegerberextensions false)
       (excludeedgelayer true)
-      (linewidth 0.100000)
+      (linewidth 2.000000)
       (plotframeref false)
-      (viasonmask false)
+      (viasonmask true)
       (mode 1)
       (useauxorigin false)
@@
       (hpglpendiameter 15)
       (hpglpenoverlay 2)
-      (psnegative false)
+      (psnegative true)
       (psa4output false)
       (plotreference true)
@@
   (net 8 "Net-(J1-Pad8)")
   (net_class Default 这是默认网络组.
-    (clearance 0.2)
-    (trace_width 0.25)
-    (via_dia 0.6)
-    (via_drill 0.4)
+    (clearance 0.25)
+    (trace_width 0.7)
+    (via_dia 0.8)
+    (via_drill 0.6)
     (uvia_dia 0.3)
     (uvia_drill 0.1)
@@
     (add_net "Net-(J1-Pad7)")
     (add_net "Net-(J1-Pad8)")
+  )
+  (module Mounting_Holes:MountingHole_3.2mm_M3 (layer F.Cu)
+    (at 112.4 127.6)
+    (descr "Mounting Hole 3.2mm, no annular, M3")
+    (tags "mounting hole 3.2mm no annular m3")
+    (fp_text reference REF** (at 0 -4.2) (layer F.SilkS)
+      (effects (font (size 1 1) (thickness 0.15)))
+    )
+    (fp_text value MountingHole_3.2mm_M3 (at 0 4.2) (layer F.Fab)
+      (effects (font (size 1 1) (thickness 0.15)))
+    )
+    (fp_circle (center 0 0) (end 3.2 0) (layer Cmts.User) (width 0.15))
+    (fp_circle (center 0 0) (end 3.45 0) (layer F.CrtYd) (width 0.05))
+    (pad 1 np_thru_hole circle (at 0 0) (size 3.2 3.2) (drill 3.2) (layers *.Cu *.Mask))
+  )
+  (module Mounting_Holes:MountingHole_3.2mm_M3 (layer F.Cu)
+    (at 112.4 100.3)
+    (descr "Mounting Hole 3.2mm, no annular, M3")
+    (tags "mounting hole 3.2mm no annular m3")
+    (fp_text reference REF** (at 0 -4.2) (layer F.SilkS)
+      (effects (font (size 1 1) (thickness 0.15)))
+    )
+    (fp_text value MountingHole_3.2mm_M3 (at 0 4.2) (layer F.Fab)
+      (effects (font (size 1 1) (thickness 0.15)))
+    )
+    (fp_circle (center 0 0) (end 3.2 0) (layer Cmts.User) (width 0.15))
+    (fp_circle (center 0 0) (end 3.45 0) (layer F.CrtYd) (width 0.05))
+    (pad 1 np_thru_hole circle (at 0 0) (size 3.2 3.2) (drill 3.2) (layers *.Cu *.Mask))
+  )
+  (module Mounting_Holes:MountingHole_3.2mm_M3 (layer F.Cu)
+    (at 152.4 100.3)
+    (descr "Mounting Hole 3.2mm, no annular, M3")
+    (tags "mounting hole 3.2mm no annular m3")
+    (fp_text reference REF** (at 0 -4.2) (layer F.SilkS)
+      (effects (font (size 1 1) (thickness 0.15)))
+    )
+    (fp_text value MountingHole_3.2mm_M3 (at 0 4.2) (layer F.Fab)
+      (effects (font (size 1 1) (thickness 0.15)))
+    )
+    (fp_circle (center 0 0) (end 3.2 0) (layer Cmts.User) (width 0.15))
+    (fp_circle (center 0 0) (end 3.45 0) (layer F.CrtYd) (width 0.05))
+    (pad 1 np_thru_hole circle (at 0 0) (size 3.2 3.2) (drill 3.2) (layers *.Cu *.Mask))
   )
   (module Pin_Headers:Pin_Header_Straight_1x08_Pitch2.54mm (layer F.Cu)
@@
     )
   )
-  (module Mounting_Holes:MountingHole_5mm (layer F.Cu)
-    (at 160.655 129.54)
-    (descr "Mounting Hole 5mm, no annular")
-    (tags "mounting hole 5mm no annular")
-    (attr virtual)
-    (fp_text reference REF** (at 0 -6) (layer F.SilkS)
-      (effects (font (size 1 1) (thickness 0.15)))
-    )
-    (fp_text value MountingHole_5mm (at 0 6) (layer F.Fab)
-      (effects (font (size 1 1) (thickness 0.15)))
-    )
-    (fp_text user %R (at 0.3 0) (layer F.Fab)
-      (effects (font (size 1 1) (thickness 0.15)))
-    )
-    (fp_circle (center 0 0) (end 5 0) (layer Cmts.User) (width 0.15))
-    (fp_circle (center 0 0) (end 5.25 0) (layer F.CrtYd) (width 0.05))
-    (pad 1 np_thru_hole circle (at 0 0) (size 5 5) (drill 5) (layers *.Cu *.Mask))
+  (module Mounting_Holes:MountingHole_3.2mm_M3 (layer F.Cu)
+    (at 152.4 127.6)
+    (descr "Mounting Hole 3.2mm, no annular, M3")
+    (tags "mounting hole 3.2mm no annular m3")
+    (fp_text reference REF** (at 0 -4.2) (layer F.SilkS)
+      (effects (font (size 1 1) (thickness 0.15)))
+    )
+    (fp_text value MountingHole_3.2mm_M3 (at 0 4.2) (layer F.Fab)
+      (effects (font (size 1 1) (thickness 0.15)))
+    )
+    (fp_circle (center 0 0) (end 3.2 0) (layer Cmts.User) (width 0.15))
+    (fp_circle (center 0 0) (end 3.45 0) (layer F.CrtYd) (width 0.05))
+    (pad 1 np_thru_hole circle (at 0 0) (size 3.2 3.2) (drill 3.2) (layers *.Cu *.Mask))
   )
   (target plus (at 112.395 100.33) (size 5) (width 0.15) (layer Edge.Cuts))
@@
   (segment (start 133.35 122.555) (end 147.32 122.555) (width 0.25) (layer F.Cu) (net 8))
   (via (at 133.35 122.555) (size 0.6) (drill 0.4) (layers F.Cu B.Cu) (net 8))
+  (zone (net 0) (net_name "") (layer F.Cu) (hatch edge 0.508)
+    (connect_pads (clearance 0.508))
+    (min_thickness 0.254)
+    (fill yes (arc_segments 16) (thermal_gap 0.508) (thermal_bridge_width 0.508))
+    (polygon
+      (pts
+        (xy 116 102.4) (xy 116 125.5) (xy 150.1 125.3) (xy 150 102.1)
+      )
+    )
+  )
+  (zone (net 0) (net_name "") (layer B.Cu) (hatch edge 0.508)
+    (connect_pads (clearance 0.508))
+    (min_thickness 0.254)
+    (fill yes (arc_segments 16) (thermal_gap 0.508) (thermal_bridge_width 0.508))
+    (polygon
+      (pts
+        (xy 149.9 125.1) (xy 116.2 125.3) (xy 116.1 102.5) (xy 116.2 102.6) (xy 149.8 102.3)
+      )
+    )
+  )
 )
